File: MTB-UNIV4.brd (EAGLE design)
At the start: 106 x 52 mm, 140 parts, among them IC1 MEGA128-A, IC2 SN75176BP, IC3 MC7805CDTG, IC4 ULN2803A, IC5 ULN2803A, X1 ARK500/2, X3 1751316, X4 1751316, X5 1751316, X6 1751316, X7 ARK500/2, X8 ARK500/2, X9 ARK500/2

Commit message: Add some GND vias.
Routing:
- net +5V: track 178.7 -> 179.2 mm
- net GND: vias 6 -> 19
Changed lines of the file:
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@@
 <via x="66.04" y="20.32" extent="1-16" drill="0.6"/>
 <via x="66.04" y="22.225" extent="1-16" drill="0.6"/>
+<via x="99.06" y="22.225" extent="1-16" drill="0.6"/>
+<via x="99.06" y="20.955" extent="1-16" drill="0.6"/>
+<via x="99.06" y="19.685" extent="1-16" drill="0.6"/>
+<via x="94.615" y="10.795" extent="1-16" drill="0.6"/>
+<via x="95.885" y="10.795" extent="1-16" drill="0.6"/>
+<via x="97.155" y="10.795" extent="1-16" drill="0.6"/>
+<via x="41.91" y="16.51" extent="1-16" drill="0.6"/>
+<via x="40.64" y="16.51" extent="1-16" drill="0.6"/>
+<via x="43.18" y="16.51" extent="1-16" drill="0.6"/>
+<via x="40.005" y="31.115" extent="1-16" drill="0.3048"/>
+<via x="40.005" y="34.29" extent="1-16" drill="0.3048"/>
+<via x="40.005" y="28.575" extent="1-16" drill="0.3048"/>
+<via x="51.435" y="23.1775" extent="1-16" drill="0.3048"/>
 </signal>
 <signal name="+5V">
@@
 <wire x1="103.1875" y1="10.7075" x2="99.11" y2="10.7075" width="1.016" layer="16"/>
 <wire x1="99.11" y1="10.7075" x2="99.06" y2="10.6575" width="1.016" layer="16"/>
-<wire x1="99.06" y1="10.6575" x2="91.7575" y2="10.6575" width="0.6096" layer="16"/>
-<wire x1="69.85" y1="17.78" x2="71.12" y2="16.51" width="0.6096" layer="16"/>
-<wire x1="69.85" y1="17.78" x2="69.85" y2="24.13" width="0.6096" layer="16"/>
-<wire x1="67.6275" y1="16.51" x2="71.12" y2="16.51" width="0.6096" layer="16"/>
+<wire x1="99.06" y1="10.6575" x2="97.79" y2="9.3875" width="0.6096" layer="16"/>
+<wire x1="97.79" y1="9.3875" x2="93.0275" y2="9.3875" width="0.6096" layer="16"/>
+<wire x1="93.0275" y1="9.3875" x2="91.7575" y2="10.6575" width="0.6096" layer="16"/>
+<wire x1="69.85" y1="16.51" x2="69.85" y2="24.13" width="0.6096" layer="16"/>
+<wire x1="67.6275" y1="16.51" x2="69.85" y2="16.51" width="0.6096" layer="16"/>
 <via x="91.7575" y="10.6575" extent="1-16" drill="0.6"/>
 <wire x1="95.25" y1="33.02" x2="93.345" y2="34.925" width="0.6096" layer="1"/>
@@
 <wire x1="79.555" y1="34.925" x2="78.74" y2="35.74" width="0.6096" layer="16"/>
 <wire x1="93.345" y1="34.925" x2="79.555" y2="34.925" width="0.6096" layer="16"/>
-<wire x1="71.12" y1="16.51" x2="85.09" y2="16.51" width="0.6096" layer="16"/>
+<wire x1="69.85" y1="16.51" x2="85.09" y2="16.51" width="0.6096" layer="16"/>
 <wire x1="91.7575" y1="10.6575" x2="90.9425" y2="10.6575" width="0.6096" layer="16"/>
 <wire x1="85.09" y1="16.51" x2="90.9425" y2="10.6575" width="0.6096" layer="16"/>
